Commit message: Add PPO training scripts and safety layer for UR3e reinforcement learning
- Implemented `train_ppo.py` for single-agent PPO training with progress tracking and model checkpointing.
- Developed `train_ppo_parallel.py` for parallel PPO training across multiple Gazebo environments, including environment management and logging.
- Created `ur3e_safety_layer` package for safety checks in reinforcement learning commands, including collision detection and joint limits.
- Added `safety_checker.py` for safety validation of joint commands and end-effector positions.
- Implemented `moveit_collision_checker.py` to publish a placeholder collision flag for integration with MoveIt.
- Established ROS node `safety_node.py` to monitor safety status based on collision and TCP pose inputs.
- Updated package configuration files for the new safety layer.

File: ur3e_rl_ws/install/ur3e_gazebo_sim/share/ur3e_gazebo_sim/urdf/ur3e_rg2_benchtop.urdf.xacro (robot description, xacro)
@@ -9,4 +9,6 @@
   <xacro:arg name="base_yaw" default="3.141592653589793"/>
   <xacro:arg name="include_rg2" default="true"/>
+  <xacro:arg name="controllers_file" default="$(find ur3e_gazebo_sim)/config/ur3e_controllers.yaml"/>
+  <xacro:arg name="initial_positions_file" default="$(find ur3e_gazebo_sim)/config/initial_positions.yaml"/>
   <xacro:arg name="joint_limits_parameters_file" default="$(find ur_description)/config/$(arg ur_type)/joint_limits.yaml"/>
   <xacro:arg name="kinematics_parameters_file" default="$(find ur_description)/config/$(arg ur_type)/default_kinematics.yaml"/>
@@ -15,4 +17,5 @@
   <xacro:include filename="$(find ur_description)/urdf/ur_macro.xacro"/>
   <xacro:include filename="$(find ur3e_gazebo_sim)/urdf/rg2_fixed.xacro"/>
+  <xacro:property name="initial_positions_file" value="$(arg initial_positions_file)"/>
   <link name="world"/>
   <xacro:ur_robot
@@ -24,5 +27,7 @@
     physical_parameters_file="$(arg physical_parameters_file)"
     visual_parameters_file="$(arg visual_parameters_file)"
-    generate_ros2_control_tag="false"
+    generate_ros2_control_tag="true"
+    sim_gazebo="true"
+    initial_positions="${xacro.load_yaml(initial_positions_file)}"
     safety_limits="true">
     <origin xyz="$(arg base_x) $(arg base_y) $(arg base_z)" rpy="0 0 $(arg base_yaw)"/>
@@ -31,3 +36,8 @@
     <xacro:rg2_fixed prefix="$(arg tf_prefix)" parent="$(arg tf_prefix)tool0"/>
   </xacro:if>
+  <gazebo>
+    <plugin filename="libgazebo_ros2_control.so" name="gazebo_ros2_control">
+      <parameters>$(arg controllers_file)</parameters>
+    </plugin>
+  </gazebo>
 </robot>
