Commit message: Fix sim launch, add approach reward, pretrained loading, cube reset, and exploration

File: ur3e_rl_ws/src/ur3e_gazebo_sim/urdf/rg2_fixed.xacro (robot description, xacro)
@@ -14,5 +14,5 @@
         <origin xyz="0 0 0" rpy="0 0 0"/>
         <geometry>
-          <mesh filename="package://ur3e_gazebo_sim/meshes/rg2/visual/${visual}.stl"/>
+          <mesh filename="$(find ur3e_gazebo_sim)/meshes/rg2/visual/${visual}.stl"/>
         </geometry>
         <material name="${name}_material">
@@ -23,5 +23,5 @@
         <origin xyz="0 0 0" rpy="0 0 0"/>
         <geometry>
-          <mesh filename="package://ur3e_gazebo_sim/meshes/rg2/collision/${collision}.stl"/>
+          <mesh filename="$(find ur3e_gazebo_sim)/meshes/rg2/collision/${collision}.stl"/>
         </geometry>
       </collision>

Commit message: working on trainig thirough providing correct joint angles for the robot is rewarded for being in to in to reach the goal. then it learns correct behaviour from that and doesnt crash into itself or spaz around as much. ran out of claude credits :(

File: ur3e_rl_ws/src/ur3e_gazebo_sim/urdf/rg2_fixed.xacro (robot description, xacro)
@@ -1,38 +1,40 @@
 <?xml version="1.0"?>
 <robot xmlns:xacro="http://wiki.ros.org/xacro">
+  <!--
+    RG2 gripper — simplified geometry.
+    The original STL files (rg2/visual/ and rg2/collision/) are corrupted and
+    cannot be parsed by Ogre3D (RViz) or ODE (Gazebo physics). Both visual and
+    collision geometry have been replaced with bounding-box approximations so
+    Gazebo can run without crashing. The kinematic chain (joint origins) is
+    unchanged, so the TCP frame and all transforms remain correct.
+  -->
   <xacro:macro name="rg2_inertial" params="mass">
     <inertial>
       <origin xyz="0 0 0" rpy="0 0 0"/>
       <mass value="${mass}"/>
-      <inertia ixx="1.0e-3" ixy="1.0e-6" ixz="1.0e-6" iyy="1.0e-3" iyz="1.0e-6" izz="1.0e-3"/>
+      <inertia ixx="1.0e-3" ixy="1.0e-6" ixz="1.0e-6"
+               iyy="1.0e-3" iyz="1.0e-6" izz="1.0e-3"/>
     </inertial>
   </xacro:macro>
-  <xacro:macro name="rg2_mesh_link" params="name visual collision rgba mass">
+  <!-- Box-approximation link: visual and collision are the same simple box -->
+  <xacro:macro name="rg2_box_link" params="name sx sy sz rgba mass">
     <link name="${name}">
       <xacro:rg2_inertial mass="${mass}"/>
       <visual>
         <origin xyz="0 0 0" rpy="0 0 0"/>
-        <geometry>
-          <mesh filename="$(find ur3e_gazebo_sim)/meshes/rg2/visual/${visual}.stl"/>
-        </geometry>
-        <material name="${name}_material">
-          <color rgba="${rgba}"/>
-        </material>
+        <geometry><box size="${sx} ${sy} ${sz}"/></geometry>
+        <material name="${name}_mat"><color rgba="${rgba}"/></material>
       </visual>
       <collision>
         <origin xyz="0 0 0" rpy="0 0 0"/>
-        <geometry>
-          <mesh filename="$(find ur3e_gazebo_sim)/meshes/rg2/collision/${collision}.stl"/>
-        </geometry>
+        <geometry><box size="${sx} ${sy} ${sz}"/></geometry>
       </collision>
     </link>
   </xacro:macro>
   <xacro:macro name="rg2_fixed" params="prefix parent">
-    <xacro:rg2_mesh_link
-      name="${prefix}onrobot_rg2_base_link"
-      visual="base_link"
-      collision="base_link"
-      rgba="0.80 0.80 0.80 1.0"
-      mass="0.78"/>
+    <!-- Gripper body -->
+    <xacro:rg2_box_link name="${prefix}onrobot_rg2_base_link"
+      sx="0.10" sy="0.08" sz="0.04"
+      rgba="0.80 0.80 0.80 1.0" mass="0.78"/>
     <joint name="${prefix}tool0-rg2_base" type="fixed">
       <parent link="${parent}"/>
@@ -40,10 +42,8 @@
       <origin xyz="0 0 0" rpy="0 0 0"/>
     </joint>
-    <xacro:rg2_mesh_link
-      name="${prefix}left_outer_knuckle"
-      visual="outer_knuckle"
-      collision="outer_knuckle"
-      rgba="0.80 0.80 0.80 1.0"
-      mass="0.05"/>
+    <!-- Left outer knuckle -->
+    <xacro:rg2_box_link name="${prefix}left_outer_knuckle"
+      sx="0.018" sy="0.018" sz="0.04"
+      rgba="0.80 0.80 0.80 1.0" mass="0.05"/>
     <joint name="${prefix}left_outer_knuckle_joint" type="fixed">
       <parent link="${prefix}onrobot_rg2_base_link"/>
@@ -51,10 +51,8 @@
       <origin xyz="0 -0.017178 0.125797" rpy="0 0 0"/>
     </joint>
-    <xacro:rg2_mesh_link
-      name="${prefix}left_inner_knuckle"
-      visual="inner_knuckle"
-      collision="inner_knuckle"
-      rgba="0.80 0.80 0.80 1.0"
-      mass="0.05"/>
+    <!-- Left inner knuckle -->
+    <xacro:rg2_box_link name="${prefix}left_inner_knuckle"
+      sx="0.014" sy="0.014" sz="0.08"
+      rgba="0.80 0.80 0.80 1.0" mass="0.05"/>
     <joint name="${prefix}left_inner_knuckle_joint" type="fixed">
       <parent link="${prefix}onrobot_rg2_base_link"/>
@@ -62,10 +60,8 @@
       <origin xyz="0 -0.007678 0.142297" rpy="0 0 0"/>
     </joint>
-    <xacro:rg2_mesh_link
-      name="${prefix}left_inner_finger"
-      visual="inner_finger"
-      collision="inner_finger"
-      rgba="0.08 0.08 0.08 1.0"
-      mass="0.05"/>
+    <!-- Left inner finger -->
+    <xacro:rg2_box_link name="${prefix}left_inner_finger"
+      sx="0.014" sy="0.014" sz="0.07"
+      rgba="0.08 0.08 0.08 1.0" mass="0.05"/>
     <joint name="${prefix}left_inner_finger_joint" type="fixed">
       <parent link="${prefix}left_outer_knuckle"/>
@@ -73,10 +69,8 @@
       <origin xyz="0 -0.039592 0.038177" rpy="0 0 0"/>
     </joint>
-    <xacro:rg2_mesh_link
-      name="${prefix}right_outer_knuckle"
-      visual="outer_knuckle"
-      collision="outer_knuckle"
-      rgba="0.80 0.80 0.80 1.0"
-      mass="0.05"/>
+    <!-- Right outer knuckle -->
+    <xacro:rg2_box_link name="${prefix}right_outer_knuckle"
+      sx="0.018" sy="0.018" sz="0.04"
+      rgba="0.80 0.80 0.80 1.0" mass="0.05"/>
     <joint name="${prefix}right_outer_knuckle_joint" type="fixed">
       <parent link="${prefix}onrobot_rg2_base_link"/>
@@ -84,10 +78,8 @@
       <origin xyz="0 0.017178 0.125797" rpy="0 0 3.141592653589793"/>
     </joint>
-    <xacro:rg2_mesh_link
-      name="${prefix}right_inner_knuckle"
-      visual="inner_knuckle"
-      collision="inner_knuckle"
-      rgba="0.80 0.80 0.80 1.0"
-      mass="0.05"/>
+    <!-- Right inner knuckle -->
+    <xacro:rg2_box_link name="${prefix}right_inner_knuckle"
+      sx="0.014" sy="0.014" sz="0.08"
+      rgba="0.80 0.80 0.80 1.0" mass="0.05"/>
     <joint name="${prefix}right_inner_knuckle_joint" type="fixed">
       <parent link="${prefix}onrobot_rg2_base_link"/>
@@ -95,10 +87,8 @@
       <origin xyz="0 0.007678 0.142297" rpy="0 0 3.141592653589793"/>
     </joint>
-    <xacro:rg2_mesh_link
-      name="${prefix}right_inner_finger"
-      visual="inner_finger"
-      collision="inner_finger"
-      rgba="0.08 0.08 0.08 1.0"
-      mass="0.05"/>
+    <!-- Right inner finger -->
+    <xacro:rg2_box_link name="${prefix}right_inner_finger"
+      sx="0.014" sy="0.014" sz="0.07"
+      rgba="0.08 0.08 0.08 1.0" mass="0.05"/>
     <joint name="${prefix}right_inner_finger_joint" type="fixed">
       <parent link="${prefix}right_outer_knuckle"/>
@@ -106,4 +96,5 @@
       <origin xyz="0 -0.039592 0.038177" rpy="0 0 0"/>
     </joint>
+    <!-- TCP frame — unchanged -->
     <link name="${prefix}gripper_tcp"/>
     <joint name="${prefix}tcp_joint" type="fixed">
